File: 考核作业/考核作业.kicad_pcb (KiCad board)
At the start: 2 copper layers, 80.7 x 104 mm, 51 parts, among them J1 USB_C_Receptacle_USB2.0, J2 Conn_01x04, J3 Conn_01x02, J4 Conn_01x19, J5 Conn_01x20, J6 Conn_01x02, J7 Conn_01x03, Q1 Q_NMOS_DGS, SW1 SW_Push, SW2 SW_Push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

Commit message: 添加敷铜
Routing:
- added copper zone on F.Cu, net (none)
Changed lines of the file:
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@@
   (segment (start 155.1406 111.89685) (end 165.2244 111.89685) (width 0.25) (layer "B.Cu") (net 57))
   (segment (start 165.2244 111.89685) (end 165.707 111.41425) (width 0.25) (layer "B.Cu") (net 57))
-  (zone (net 0) (net_name "") (layer "Edge.Cuts") (hatch edge 0.508)
-    (connect_pads (clearance 0.508))
+  (zone (net 0) (net_name "") (layer "F.Cu") (hatch edge 0.508)
+    (connect_pads yes (clearance 0.508))
     (min_thickness 0.254) (filled_areas_thickness no)
     (fill yes (thermal_gap 0.508) (thermal_bridge_width 0.508))
     (polygon
       (pts
-        (xy 191.4906 27.813)
-        (xy 191.262 131.8514)
-        (xy 109.855 131.3942)
-        (xy 109.8804 27.7114)
+        (xy 191.1096 27.7368)
+        (xy 191.1096 131.8768)
+        (xy 110.2614 131.8768)
+        (xy 110.236 27.686)
       )
     )
